Commit message: test: isolate runtime and prove RTX invalid ranges are ambiguous

File: config/generated/jackal.urdf (robot description, URDF)
Before this commit: robot jackal, 14 links, 13 joints
Links:
- link chassis_link: geometry collision box size=0.42 0.31 0.184; visual mesh filename=/home/lpc/workspace/arena5_ws_costmap_fix/src/arena/simulat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
- link front_fender_link: geometry visual mesh filename=/home/lpc/workspace/arena5_ws_costmap_fix/src/arena/simulat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
- link front_left_wheel_link: geometry collision cylinder length=0.04 radius=0.098; visual mesh filename=/home/lpc/workspace/arena5_ws_costmap_fix/src/arena/simulat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
- link front_right_wheel_link: geometry collision cylinder length=0.04 radius=0.098; visual mesh filename=/home/lpc/workspace/arena5_ws_costmap_fix/src/arena/simulat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
- link rear_fender_link: geometry visual mesh filename=/home/lpc/workspace/arena5_ws_costmap_fix/src/arena/simulat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
- link rear_left_wheel_link: geometry collision cylinder length=0.04 radius=0.098; visual mesh filename=/home/lpc/workspace/arena5_ws_costmap_fix/src/arena/simulat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
- link rear_right_wheel_link: geometry collision cylinder length=0.04 radius=0.098; visual mesh filename=/home/lpc/workspace/arena5_ws_costmap_fix/src/arena/simulat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
